Commit message: naprawa3

File: src/ros2_RobotSimulation/Cyton/cyton_ros2_gazebo/urdf/cyton_gazebo.xacro (robot description, xacro)
@@ -164,5 +164,5 @@
       </joint>
       <!-- cyton_finger_joint1 -->
-      <joint name="gripper_joint">
+      <!-- <joint name="gripper_joint">
         <command_interface name="position">
           <param name="min">-0.001</param>
@@ -176,7 +176,7 @@
         <state_interface name="velocity"/>
         <state_interface name="effort"/>
-      </joint>
+      </joint> -->
       <!-- cyton_finger_joint2 -->
-      <joint name="gripper_joint2">
+      <!-- <joint name="gripper_joint2">
         <command_interface name="position">
           <param name="min">-0.001</param>
@@ -190,5 +190,5 @@
         <state_interface name="velocity"/>
         <state_interface name="effort"/>
-      </joint>
+      </joint> -->
     </ros2_control>
     <gazebo reference="shoulder_roll">
@@ -220,5 +220,5 @@
       <material>Gazebo/Orange</material>
     </gazebo>
-    <gazebo reference="gripper_finger1">
+    <!-- <gazebo reference="gripper_finger1">
       <selfCollide>false</selfCollide>
       <material>Gazebo/Orange</material>
@@ -231,5 +231,5 @@
       <selfCollide>false</selfCollide>
       <material>Gazebo/Orange</material>
-    </gazebo>
+    </gazebo> -->
     <gazebo reference="base_footprint">
       <selfCollide>false</selfCollide>
@@ -240,9 +240,9 @@
       <material>Gazebo/Orange</material>
     </gazebo>
-    <gazebo reference="virtual_endeffector_joint">
-      <preserveFixedJoint>true</preserveFixedJoint>
+    <!-- <gazebo reference="virtual_endeffector_joint">
+      <preserveFixedJoint>true</preserveFixedJoint> -->
       <!-- For compatibility with SDFormat < 4.4 -->
-      <disableFixedJointLumping>true</disableFixedJointLumping>
-    </gazebo>
+      <!-- <disableFixedJointLumping>true</disableFixedJointLumping>
+    </gazebo> -->
   </xacro:macro>
 </robot>

File: src/ros2_RobotSimulation/Cyton/cyton_ros2_gazebo/urdf/cyton_macros.urdf.xacro (robot description, xacro)
@@ -30,5 +30,5 @@
                 <origin xyz="0 0 0" rpy="0 0 0" />
                 <geometry>
-                    <mesh filename="package://cyton_ros2_gazebo/meshes/gamma_base.dae" />
+                    <mesh filename="file://$(find cyton_ros2_gazebo)/meshes/visual/gamma_base.dae" />
                 </geometry>
             </visual>
@@ -58,5 +58,5 @@
                 <origin xyz="0 0 0" rpy="1.5708 0 3.14159" />
                 <geometry>
-                    <mesh filename="package://cyton_ros2_gazebo/meshes/Shoulder_Roll.dae" />
+                    <mesh filename="file://$(find cyton_ros2_gazebo)/meshes/visual/Shoulder_Roll.dae" />
                 </geometry>
             </visual>
@@ -86,5 +86,5 @@
                 <origin xyz="0.028 0 0" rpy="0 1.5708 0" />
                 <geometry>
-                    <mesh filename="package://cyton_ros2_gazebo/meshes/Shoulder_Pitch.dae" />
+                    <mesh filename="file://$(find cyton_ros2_gazebo)/meshes/visual/Shoulder_Pitch.dae" />
                 </geometry>
             </visual>
@@ -114,5 +114,5 @@
                 <origin xyz="0 0 0" rpy="0 0 3.92699" />
                 <geometry>
-                    <mesh filename="package://cyton_ros2_gazebo/meshes/Elbow_Roll.dae" />
+                    <mesh filename="file://$(find cyton_ros2_gazebo)/meshes/visual/Elbow_Roll.dae" />
                 </geometry>
             </visual>
@@ -143,5 +143,5 @@
                 <origin xyz="0.027 0 0" rpy="1.5708 0 1.5708" />
                 <geometry>
-                    <mesh filename="package://cyton_ros2_gazebo/meshes/Elbow_Pitch.dae" />
+                    <mesh filename="file://$(find cyton_ros2_gazebo)/meshes/visual/Elbow_Pitch.dae" />
                 </geometry>
             </visual>
@@ -171,5 +171,5 @@
                 <origin xyz="0 0 0" rpy="1.5708 0 0" />
                 <geometry>
-                    <mesh filename="package://cyton_ros2_gazebo/meshes/Elbow_Yaw.dae" />
+                    <mesh filename="file://$(find cyton_ros2_gazebo)/meshes/visual/Elbow_Yaw.dae" />
                 </geometry>
             </visual>
@@ -199,5 +199,5 @@
                 <origin xyz="0.027 0 0" rpy="1.5708 0 1.5708" />
                 <geometry>
-                    <mesh filename="package://cyton_ros2_gazebo/meshes/Wrist_Pitch.dae" />
+                    <mesh filename="file://$(find cyton_ros2_gazebo)/meshes/visual/Wrist_Pitch.dae" />
                 </geometry>
             </visual>
@@ -227,5 +227,5 @@
                 <origin xyz="0 0 0" rpy="0 3.14159 1.5708" />
                 <geometry>
-                    <mesh filename="package://cyton_ros2_gazebo/meshes/Wrist_Roll.dae" />
+                    <mesh filename="file://$(find cyton_ros2_gazebo)/meshes/visual/Wrist_Roll.dae" />
                 </geometry>
             </visual>
@@ -255,5 +255,5 @@
                 <origin xyz="0 0 0" rpy="0 0 0" />
                 <geometry>
-                    <mesh filename="package://cyton_ros2_gazebo/meshes/Gripper_Finger1.dae"/>
+                    <mesh filename="file://$(find cyton_ros2_gazebo)/meshes/visual/Gripper_Finger1.dae"/>
                 </geometry>
             </visual>
@@ -278,5 +278,5 @@
                 <origin xyz="0 0 0" rpy="0 0 0" />
                 <geometry>
-                    <mesh filename="package://cyton_ros2_gazebo/meshes/Gripper_Finger2.dae"/>
+                    <mesh filename="file://$(find cyton_ros2_gazebo)/meshes/visual/Gripper_Finger2.dae"/>
                 </geometry>
             </visual>
