Commit message: Koniec padaczki

File: src/ros2_RobotSimulation/Cyton/cyton_ros2_gazebo/urdf/cyton.urdf.xacro (robot description, xacro)
@@ -10,5 +10,5 @@
     <!-- <child link = "panda_base" /> -->
     <child link = "base_link" />
-    <origin xyz="0.0 0.0 0.0" rpy="0.0 0.0 0.0" /> <!-- <origin xyz="0.0 0.0 0.65" rpy="0.0 0.0 0.0" /> -->
+    <origin xyz="0.0 0.0 0.65" rpy="0.0 0.0 0.0" /> <!-- <origin xyz="0.0 0.0 0.65" rpy="0.0 0.0 0.0" /> -->
   </joint>
 </robot>

File: src/ros2_RobotSimulation/Cyton/cyton_ros2_gazebo/urdf/cyton_macros.urdf.xacro (robot description, xacro)
@@ -7,8 +7,15 @@
         <xacro:cyton_gazebo />
         <!-- Initial footprint motor used here -->
-        <xacro:macro name="base_footprint" params="prefix">
+        <xacro:macro name="base_footprint">
             <link name="base_footprint">
+                <!-- ZMIENIĆ!!! -->
+                <inertial>
+                    <mass value="2.92"/>
+                    <origin rpy="0 0 0" xyz="-0.025566 -2.88e-05 0.057332"/>
+                    <inertia ixx="0.00782229414331" ixy="-1.56191622996e-05" ixz="-0.00126005738123" iyy="0.0109027971813" iyz="1.08233858202e-05" izz="0.0102355503949"/>
+                  </inertial>
+                <!-- ZMIENIĆ -->
                 <visual>
-                    <origin xyz="0 0 0" rpy="0 0 0" />
+                    <origin xyz="0 0 1" rpy="0 0 0" />
                     <geometry>
                         <sphere radius="0.001" />
@@ -18,8 +25,15 @@
                     </material>
                 </visual>
+                <collision>
+                    <origin xyz="0 0 0" rpy="0 0 0" />
+                    <geometry>
+                        <sphere radius="0.001" />
+                    </geometry>
+                </collision>
             </link>
             <joint name="base_joint" type="fixed">
                 <parent link="base_footprint" />
                 <child link="base_link" />
+                <dynamics damping="0.5" friction="0.5"/>
                 <origin xyz="0.0 0.0 0.0" rpy="0 0 0" />
             </joint>
@@ -36,5 +50,5 @@
                 <origin xyz="0 0.0115 0.047" />
                 <geometry>
-                    <box size="0.154 0.177 0.094" />
+                    <box size="0.01 0.01 0.01" />
                 </geometry>
             </collision>
@@ -43,5 +57,5 @@
                 <origin rpy="0 0 0" xyz="0 0 0" />
                 <inertia ixx="1.1027" iyy="1.1027" izz="1.1027"
-                    ixy="0" ixz="0" iyz="0" />
+                    ixy="0.05" ixz="0.05" iyz="0.05" />
             </inertial>
         </link>
@@ -51,5 +65,6 @@
             <child link="shoulder_roll" />
             <origin xyz="0 0 0.05315" rpy="0 0 1.2" />
-            <limit lower="-2.618" upper="2.618" effort="100.0" velocity="1.0" />
+            <dynamics damping="0.5" friction="0.5"/>
+            <limit lower="-2.618" upper="2.618" effort="7.0" velocity="1.0" />
             <axis xyz="0 0 1" />
         </joint>
@@ -71,5 +86,5 @@
                 <origin rpy="0 0 0" xyz="0 0 0" />
                 <inertia ixx=".1027" iyy=".1027" izz=".1027"
-                    ixy="0" ixz="0" iyz="0" />
+                    ixy="0.05" ixz="0.05" iyz="0.05" />
             </inertial>
         </link>
@@ -79,5 +94,6 @@
             <child link="shoulder_pitch" />
             <origin xyz="0 0 0.063" rpy="1.2 0 0" />
-            <limit lower="-1.8326" upper="1.8326" effort="100.0" velocity="1.0" />
+            <dynamics damping="0.5" friction="0.5"/>
+            <limit lower="-1.8326" upper="1.8326" effort="7.0" velocity="1.0" />
             <axis xyz="1 0 0" />
         </joint>
@@ -99,7 +115,8 @@
                 <origin rpy="0 0 0" xyz="0 0 0" />
                 <inertia ixx=".0827" iyy=".0827" izz=".0827"
-                    ixy="0" ixz="0" iyz="0" />
-            </inertial>
-        </link>
+                    ixy="0.05" ixz="0.05" iyz="0.05" />
+            </inertial>
+        </link>
+<!-- TUTAJ ODPIERDALA -->
         <!-- Third motor located here -->
         <joint name="elbow_roll_joint" type="revolute">
@@ -107,5 +124,6 @@
             <child link="elbow_roll" />
             <origin xyz="0 0 0.089" rpy="0 0 1.2" />
-            <limit lower="-1.8326" upper="1.8326" effort="100.0" velocity="1.0" />
+            <dynamics damping="0.5" friction="0.5"/>
+            <limit lower="-1.8326" upper="1.8326" effort="7.0" velocity="1.0" />
             <axis xyz="0 0 1" />
         </joint>
@@ -127,5 +145,5 @@
                 <origin rpy="0 0 0" xyz="0 0 0" />
                 <inertia ixx=".0627" iyy=".0627" izz=".0627"
-                    ixy="0" ixz="0" iyz="0" />
+                    ixy="0.05" ixz="0.05" iyz="0.05" />
             </inertial>
         </link>
@@ -135,5 +153,6 @@
             <child link="elbow_pitch" />
             <origin xyz="0 0 0.052" rpy="1.2 0 0" />
-            <limit lower="-1.8326" upper="1.8326" effort="100.0" velocity="1.0" />
+            <dynamics damping="0.5" friction="0.5"/>
+            <limit lower="-1.8326" upper="1.8326" effort="7.0" velocity="1.0" />
             <axis xyz="1 0 0" />
         </joint>
@@ -156,5 +175,5 @@
                 <origin rpy="0 0 0" xyz="0 0 0" />
                 <inertia ixx=".0327" iyy=".0327" izz=".0327"
-                    ixy="0" ixz="0" iyz="0" />
+                    ixy="0.05" ixz="0.05" iyz="0.05" />
             </inertial>
         </link>
@@ -164,5 +183,6 @@
             <child link="elbow_yaw" />
             <origin xyz="0 0 0.072" rpy="0 -1.2 0" />
-            <limit lower="-1.8326" upper="1.8326" effort="100.0" velocity="1.0" />
+            <dynamics damping="0.5" friction="0.5"/>
+            <limit lower="-1.8326" upper="1.8326" effort="7.0" velocity="1.0" />
             <axis xyz="0 -1 0" />
         </joint>
@@ -184,5 +204,5 @@
                 <origin rpy="0 0 0" xyz="0 0 0" />
                 <inertia ixx=".0227" iyy=".0227" izz=".0227"
-                    ixy="0" ixz="0" iyz="0" />
+                    ixy="0.05" ixz="0.05" iyz="0.05" />
             </inertial>
         </link>
@@ -192,5 +212,6 @@
             <child link="wrist_pitch" />
             <origin xyz="0 0 0.0718" rpy="1.2 0 0" />
-            <limit lower="-1.8326" upper="1.8326" effort="100.0" velocity="1.0" />
+            <dynamics damping="0.5" friction="0.5"/>
+            <limit lower="-1.8326" upper="1.8326" effort="7.0" velocity="1.0" />
             <axis xyz="1 0 0" />
         </joint>
@@ -212,5 +233,5 @@
                 <origin rpy="0 0 0" xyz="0 0 0" />
                 <inertia ixx=".0127" iyy=".0127" izz=".0127"
-                    ixy="0" ixz="0" iyz="0" />
+                    ixy="0.05" ixz="0.05" iyz="0.05" />
             </inertial>
         </link>
@@ -220,5 +241,6 @@
             <child link="wrist_roll" />
             <origin xyz="0 0 0.051425" rpy="0 0 1.2" />
-            <limit lower="-2.61799" upper="2.61799" effort="100.0" velocity="1.0" />
+            <dynamics damping="0.5" friction="0.5"/>
+            <limit lower="-2.61799" upper="2.61799" effort="7.0" velocity="1.0" />
             <axis xyz="0 0 1" />
         </joint>
@@ -240,5 +262,5 @@
                 <origin rpy="0 0 0" xyz="0 0 0" />
                 <inertia ixx=".0027" iyy=".0027" izz=".0027"
-                    ixy="0" ixz="0" iyz="0" />
+                    ixy="0.05" ixz="0.05" iyz="0.05" />
             </inertial>
         </link>
@@ -248,5 +270,5 @@
             <child link="gripper_finger1" />
             <origin xyz="-0.01331 0.00485 0.077225" rpy="0 0 0" />
-            <limit lower="-0.008" upper="0.008" effort="100.0" velocity="1.0" />
+            <limit lower="-0.008" upper="0.008" effort="7.0" velocity="1.0" />
             <axis xyz="1 0 0" />
         </joint>
@@ -270,5 +292,5 @@
             <child link="gripper_finger2" />
             <origin xyz="0.0098 0.00485 0.077225" rpy="0 0 0" />
-            <limit lower="-0.008" upper="0.008" effort="100.0" velocity="1.0" />
+            <limit lower="-0.008" upper="0.008" effort="7.0" velocity="1.0" />
             <mimic joint="gripper_joint" multiplier="-1"/>
             <axis xyz="1 0 0" />

Commit message: Naprawic kolizje w URDF

File: src/ros2_RobotSimulation/Cyton/cyton_ros2_gazebo/urdf/cyton.urdf.xacro (robot description, xacro)
@@ -8,7 +8,6 @@
   <joint name="world_joint" type="fixed">
     <parent link="world" />
-    <!-- <child link = "panda_base" /> -->
     <child link = "base_link" />
-    <origin xyz="0.0 0.0 0.65" rpy="0.0 0.0 0.0" /> <!-- <origin xyz="0.0 0.0 0.65" rpy="0.0 0.0 0.0" /> -->
+    <origin xyz="0.0 0.0 0.01" rpy="0.0 0.0 0.0" />
   </joint>
 </robot>

File: src/ros2_RobotSimulation/Cyton/cyton_ros2_gazebo/urdf/cyton_macros.urdf.xacro (robot description, xacro)
@@ -26,7 +26,7 @@
                 </visual>
                 <collision>
-                    <origin xyz="0 0 0" rpy="0 0 0" />
+                    <origin xyz="0 0 1" rpy="0 0 0" />
                     <geometry>
-                        <sphere radius="0.001" />
+                        <sphere radius="0.01" />
                     </geometry>
                 </collision>
@@ -47,10 +47,22 @@
                 </geometry>
             </visual>
-            <collision>
+            <!-- <collision>
                 <origin xyz="0 0.0115 0.047" />
                 <geometry>
                     <box size="0.01 0.01 0.01" />
                 </geometry>
-            </collision>
+            </collision> -->
+            <collision>
+                <origin xyz="0 0 0.0026" />
+                <geometry>
+                    <box size="0.1 0.1 0.007" />
+                </geometry>
+            </collision>
+            <!-- <collision>
+                <origin xyz="0 0 0" rpy="0 0 0" />
+                <geometry>
+                    <sphere radius="0.001" />
+                </geometry>
+            </collision> -->
             <inertial>
                 <mass value="100.0" />
@@ -76,8 +88,20 @@
                 </geometry>
             </visual>
-            <collision>
+            <!-- <collision>
                 <origin xyz="0.0 0.069 0.0587" />
                 <geometry>
                     <box size="0.09829 0.18143 0.08392" />
+                </geometry>
+            </collision> -->
+            <!-- <collision>
+                <origin xyz="0 0 0" />
+                <geometry>
+                    <box size="0.09829 0.18143 0.08392" />
+                </geometry>
+            </collision> -->
+            <collision>
+                <origin xyz="0 0 0" rpy="0 0 0" />
+                <geometry>
+                    <sphere radius="0.001" />
                 </geometry>
             </collision>
@@ -105,8 +129,20 @@
                 </geometry>
             </visual>
-            <collision>
+            <!-- <collision>
                 <origin xyz="-0.001 0.064 0.1745" />
                 <geometry>
                     <box size="0.0709 0.19363 0.083" />
+                </geometry>
+            </collision> -->
+            <!-- <collision>
+                <origin xyz="0.028 0 0" />
+                <geometry>
+                    <box size="0.0709 0.19363 0.083" />
+                </geometry>
+            </collision> -->
+            <collision>
+                <origin xyz="0 0 0" rpy="0 0 0" />
+                <geometry>
+                    <sphere radius="0.001" />
                 </geometry>
             </collision>
@@ -135,8 +171,20 @@
                 </geometry>
             </visual>
-            <collision>
+            <!-- <collision>
                 <origin xyz="-0.0225 0.039 0.3068" />
                 <geometry>
                     <box size="0.0717 0.1846 0.0756" />
+                </geometry>
+            </collision> -->
+            <!-- <collision>
+                <origin xyz="0 0 0" />
+                <geometry>
+                    <box size="0.0717 0.1846 0.0756" />
+                </geometry>
+            </collision> -->
+            <collision>
+                <origin xyz="0 0 0" rpy="0 0 0" />
+                <geometry>
+                    <sphere radius="0.001" />
                 </geometry>
             </collision>
@@ -165,8 +213,20 @@
                 </geometry>
             </visual>
-            <collision>
+            <!-- <collision>
                 <origin xyz="0.0346 0.0461 0.4228" />
                 <geometry>
                     <box size="0.0549 0.1557 0.076" />
+                </geometry>
+            </collision> -->
+            <!-- <collision>
+                <origin xyz="0.027 0 0" />
+                <geometry>
+                    <box size="0.0549 0.1557 0.076" />
+                </geometry>
+            </collision> -->
+            <collision>
+                <origin xyz="0 0 0" rpy="0 0 0" />
+                <geometry>
+                    <sphere radius="0.001" />
                 </geometry>
             </collision>
@@ -194,8 +254,20 @@
                 </geometry>
             </visual>
-            <collision>
+            <!-- <collision>
                 <origin xyz="0.0172 0.0209 0.516" />
                 <geometry>
                     <box size="0.0535 0.1160 0.0402" />
+                </geometry>
+            </collision> -->
+            <!-- <collision>
+                <origin xyz="0 0 0" />
+                <geometry>
+                    <box size="0.0535 0.1160 0.0402" />
+                </geometry>
+            </collision> -->
+            <collision>
+                <origin xyz="0 0 0" rpy="0 0 0" />
+                <geometry>
+                    <sphere radius="0.001" />
                 </geometry>
             </collision>
@@ -223,8 +295,20 @@
                 </geometry>
             </visual>
-            <collision>
+            <!-- <collision>
                 <origin xyz="0.0257 0.0118 0.5617" />
                 <geometry>
                     <box size="0.026 0.0435 0.05185" />
+                </geometry>
+            </collision> -->
+            <!-- <collision>
+                <origin xyz="0.027 0 0" />
+                <geometry>
+                    <box size="0.026 0.0435 0.05185" />
+                </geometry>
+            </collision> -->
+            <collision>
+                <origin xyz="0 0 0" rpy="0 0 0" />
+                <geometry>
+                    <sphere radius="0.001" />
                 </geometry>
             </collision>
@@ -252,8 +336,20 @@
                 </geometry>
             </visual>
-            <collision>
+            <!-- <collision>
                 <origin xyz="-0.0063 -0.0014 0.6102" />
                 <geometry>
                     <box size="0.0518 0.0723 0.1004" />
+                </geometry>
+            </collision> -->
+            <!-- <collision>
+                <origin xyz="0 0 0" />
+                <geometry>
+                    <box size="0.0518 0.0723 0.1004" />
+                </geometry>
+            </collision> -->
+            <collision>
+                <origin xyz="0 0 0" rpy="0 0 0" />
+                <geometry>
+                    <sphere radius="0.001" />
                 </geometry>
             </collision>
